File: usb_serial/usb_serial.kicad_sch (KiCad schematic)
At the start: 3 parts, among them J1 47589-1001, J3 Conn_01x04_Pin, U1 FT232RL

Commit message: Power+Decoupling
Parts:
- added C1: 10n, Capacitor_SMD:C_0402_1005Metric, symbol Device:C_Small
- added C2: 4.7u, Capacitor_SMD:C_0805_2012Metric, symbol Device:C_Small
- added C3, C4: 100n, Capacitor_SMD:C_0402_1005Metric, symbol Device:C_Small
Connections:
- net +3.3V: now reaches U1.17 (3V3OUT)
- net +3.3V: now also U1.4 (VCCIO), C4.1
- net GND: now reaches U1.18 (GND)
- net GND: now also J1.5 (GND), J1.SH1 (SHIELD), J1.SH2 (SHIELD), J1.SH3 (SHIELD), J1.SH4 (SHIELD), J1.SH5 (SHIELD), J1.SH6 (SHIELD), J3.4 (Pin_4), U1.21 (GND), U1.25 (AGND), U1.26 (TEST), U1.7 (GND), C1.2, C2.2, C3.2, C4.2
- net +5V: now reaches U1.20 (VCC)
- net +5V: now also J1.1 (VBUS), J3.1 (Pin_1), C1.1, C2.1, C3.1
Other:
- moved on the sheet: J1, J3, U1

Commit message: Schematic complete
Parts:
- added D1, D2, D3: LED, LED_SMD:LED_0805_2012Metric, symbol Device:LED
- added R1, R2: 1k, Resistor_SMD:R_0402_1005Metric, symbol Device:R_Small_US
- added R3: 2.2k, Resistor_SMD:R_0402_1005Metric, symbol Device:R_Small_US
Connections:
- net +3.3V: now also D1.2 (A), D2.2 (A)
- net +5V: now also D3.2 (A)
- net GND: now also R3.1
- net UART_TX: now reaches U1.1 (TXD)
- net UART_TX: now also J3.2 (Pin_2), R1.1
- net USB_DP: now reaches U1.15 (USBDP)
- net USB_DP: now also J1.3 (D+)
- net USB_DN: now reaches U1.16 (USBDM)
- net USB_DN: now also J1.2 (D-)
- net UART_RX: now reaches U1.5 (RXD)
- net UART_RX: now also J3.3 (Pin_3), R2.1
- new net: D3.1 (K), R3.2
- new net: D1.1 (K), R1.2
- new net: D2.1 (K), R2.2
- no-connect marks 0 -> 15
Other:
- moved on the sheet: C2, C3, C4, J3, U1
